File: pcb/yosino58.sch (KiCad schematic (older format))
At the start: 110 parts, among them J0 LED, J1 TRRS, J2 OLED, J3 OLED, J4 OLED, J5 OLED, J6 OLED, P1 i2c_pin, P2 i2c_pin, SW1 SW_PUSH, SW10 SW_PUSH, SW11 SW_PUSH, SW12 SW_PUSH, SW13 SW_PUSH, SW14 SW_PUSH, SW15 SW_PUSH, SW16 SW_PUSH, SW17 SW_PUSH, SW18 SW_PUSH, SW19 SW_PUSH, SW2 SW_PUSH, SW20 SW_PUSH, SW21 SW_PUSH, SW22 SW_PUSH, SW23 SW_PUSH, SW24 SW_PUSH, SW25 SW_PUSH, SW26 SW_PUSH, SW27 SW_PUSH, SW28 SW_PUSH, SW29 SW_PUSH, SW3 SW_PUSH, SW4 SW_PUSH, SW5 SW_PUSH, SW6 SW_PUSH, SW7 SW_PUSH, SW8 SW_PUSH, SW9 SW_PUSH, U1 ProMicro, U2 ProMicro

Commit message: SK6812MINIの外形修正
Parts:
- J1: symbol yosino58-rescue:MJ-4PP-9-kbd-yosino58-rescue -> yosino58-rescue:MJ-4PP
- L1, L10, L11, L12, L13, L14, L15, L16, L17, L18, L19, L2, L20, L21, L22, L23, L24, L25, L26, L27, L28, L29, L3, L4, L5, L6, L7, L8, L9: symbol yosino58-rescue:SK6812MINI-kbd-yosino58-rescue -> yosino58-rescue:SK6812MINI
- RSW1, SW1, SW10, SW11, SW12, SW13, SW14, SW15, SW16, SW17, SW18, SW19, SW2, SW20, SW21, SW22, SW23, SW24, SW25, SW26, SW27, SW28, SW29, SW3, SW4, SW5, SW6, SW7, SW8, SW9: symbol yosino58-rescue:SW_PUSH-kbd-yosino58-rescue -> yosino58-rescue:SW_PUSH
- U1, U2: symbol yosino58-rescue:ProMicro-kbd-yosino58-rescue -> yosino58-rescue:ProMicro-BLE
Changed lines of the file:
@@
 $EndDescr
 $Comp
-L yosino58-rescue:ProMicro-kbd-yosino58-rescue U1
+L yosino58-rescue:ProMicro-BLE U1
 U 1 1 5C510A34
 P 2325 1675
@@
 $EndComp
 $Comp
-L yosino58-rescue:SW_PUSH-kbd-yosino58-rescue SW7
+L yosino58-rescue:SW_PUSH SW7
 U 1 1 5C510E26
 P 7250 1425
@@
 $EndComp
 $Comp
-L yosino58-rescue:SW_PUSH-kbd-yosino58-rescue SW8
+L yosino58-rescue:SW_PUSH SW8
 U 1 1 5C5116E3
 P 7950 1425
@@
 $EndComp
 $Comp
-L yosino58-rescue:SW_PUSH-kbd-yosino58-rescue SW9
+L yosino58-rescue:SW_PUSH SW9
 U 1 1 5C511809
 P 8650 1425
@@
 $EndComp
 $Comp
-L yosino58-rescue:SW_PUSH-kbd-yosino58-rescue SW10
+L yosino58-rescue:SW_PUSH SW10
 U 1 1 5C511817
 P 9350 1425
@@
 $EndComp
 $Comp
-L yosino58-rescue:SW_PUSH-kbd-yosino58-rescue SW11
+L yosino58-rescue:SW_PUSH SW11
 U 1 1 5C51197C
 P 10050 1425
@@
 $EndComp
 $Comp
-L yosino58-rescue:SW_PUSH-kbd-yosino58-rescue SW12
+L yosino58-rescue:SW_PUSH SW12
 U 1 1 5C51198A
 P 10750 1425
@@
 $EndComp
 $Comp
-L yosino58-rescue:SW_PUSH-kbd-yosino58-rescue SW1
+L yosino58-rescue:SW_PUSH SW1
 U 1 1 5C511EAC
 P 7250 925
@@
 $EndComp
 $Comp
-L yosino58-rescue:SW_PUSH-kbd-yosino58-rescue SW2
+L yosino58-rescue:SW_PUSH SW2
 U 1 1 5C511EBA
 P 7950 925
@@
 $EndComp
 $Comp
-L yosino58-rescue:SW_PUSH-kbd-yosino58-rescue SW3
+L yosino58-rescue:SW_PUSH SW3
 U 1 1 5C511EC8
 P 8650 925
@@
 $EndComp
 $Comp
-L yosino58-rescue:SW_PUSH-kbd-yosino58-rescue SW4
+L yosino58-rescue:SW_PUSH SW4
 U 1 1 5C511ED6
 P 9350 925
@@
 $EndComp
 $Comp
-L yosino58-rescue:SW_PUSH-kbd-yosino58-rescue SW5
+L yosino58-rescue:SW_PUSH SW5
 U 1 1 5C511EE4
 P 10050 925
@@
 $EndComp
 $Comp
-L yosino58-rescue:SW_PUSH-kbd-yosino58-rescue SW6
+L yosino58-rescue:SW_PUSH SW6
 U 1 1 5C511EF2
 P 10750 925
@@
 $EndComp
 $Comp
-L yosino58-rescue:SW_PUSH-kbd-yosino58-rescue SW13
+L yosino58-rescue:SW_PUSH SW13
 U 1 1 5C51227A
 P 7250 1925
@@
 $EndComp
 $Comp
-L yosino58-rescue:SW_PUSH-kbd-yosino58-rescue SW14
+L yosino58-rescue:SW_PUSH SW14
 U 1 1 5C512288
 P 7950 1925
@@
 $EndComp
 $Comp
-L yosino58-rescue:SW_PUSH-kbd-yosino58-rescue SW15
+L yosino58-rescue:SW_PUSH SW15
 U 1 1 5C512296
 P 8650 1925
@@
 $EndComp
 $Comp
-L yosino58-rescue:SW_PUSH-kbd-yosino58-rescue SW16
+L yosino58-rescue:SW_PUSH SW16
 U 1 1 5C5122A4
 P 9350 1925
@@
 $EndComp
 $Comp
-L yosino58-rescue:SW_PUSH-kbd-yosino58-rescue SW17
+L yosino58-rescue:SW_PUSH SW17
 U 1 1 5C5122B2
 P 10050 1925
@@
 $EndComp
 $Comp
-L yosino58-rescue:SW_PUSH-kbd-yosino58-rescue SW18
+L yosino58-rescue:SW_PUSH SW18
 U 1 1 5C5122C0
 P 10750 1925
@@
 $EndComp
 $Comp
-L yosino58-rescue:SW_PUSH-kbd-yosino58-rescue SW19
+L yosino58-rescue:SW_PUSH SW19
 U 1 1 5C512594
 P 7250 2425
@@
 $EndComp
 $Comp
-L yosino58-rescue:SW_PUSH-kbd-yosino58-rescue SW20
+L yosino58-rescue:SW_PUSH SW20
 U 1 1 5C5125A2
 P 7950 2425
@@
 $EndComp
 $Comp
-L yosino58-rescue:SW_PUSH-kbd-yosino58-rescue SW21
+L yosino58-rescue:SW_PUSH SW21
 U 1 1 5C5125B0
 P 8650 2425
@@
 $EndComp
 $Comp
-L yosino58-rescue:SW_PUSH-kbd-yosino58-rescue SW22
+L yosino58-rescue:SW_PUSH SW22
 U 1 1 5C5125BE
 P 9350 2425
@@
 $EndComp
 $Comp
-L yosino58-rescue:SW_PUSH-kbd-yosino58-rescue SW23
+L yosino58-rescue:SW_PUSH SW23
 U 1 1 5C5125CC
 P 10050 2425
@@
 $EndComp
 $Comp
-L yosino58-rescue:SW_PUSH-kbd-yosino58-rescue SW24
+L yosino58-rescue:SW_PUSH SW24
 U 1 1 5C5125DA
 P 10750 2425
@@
 	10350 1225 11050 1225
 $Comp
-L yosino58-rescue:SW_PUSH-kbd-yosino58-rescue SW25
+L yosino58-rescue:SW_PUSH SW25
 U 1 1 5C51A620
 P 7950 2925
@@
 $EndComp
 $Comp
-L yosino58-rescue:SW_PUSH-kbd-yosino58-rescue SW26
+L yosino58-rescue:SW_PUSH SW26
 U 1 1 5C51A62E
 P 8650 2925
@@
 $EndComp
 $Comp
-L yosino58-rescue:SW_PUSH-kbd-yosino58-rescue SW27
+L yosino58-rescue:SW_PUSH SW27
 U 1 1 5C51A63C
 P 9350 2925
@@
 $EndComp
 $Comp
-L yosino58-rescue:SW_PUSH-kbd-yosino58-rescue SW28
+L yosino58-rescue:SW_PUSH SW28
 U 1 1 5C51A64A
 P 10050 2925
@@
 $EndComp
 $Comp
-L yosino58-rescue:SW_PUSH-kbd-yosino58-rescue SW29
+L yosino58-rescue:SW_PUSH SW29
 U 1 1 5C51A658
 P 10750 2925
@@
 SCL
 $Comp
-L yosino58-rescue:MJ-4PP-9-kbd-yosino58-rescue J1
+L yosino58-rescue:MJ-4PP J1
 U 1 1 5C558952
 P 4700 3325
@@
 $EndComp
 $Comp
-L yosino58-rescue:SK6812MINI-kbd-yosino58-rescue L6
+L yosino58-rescue:SK6812MINI L6
 U 1 1 5C558DB2
 P 9675 4025
@@
 $EndComp
 $Comp
-L yosino58-rescue:SK6812MINI-kbd-yosino58-rescue L5
+L yosino58-rescue:SK6812MINI L5
 U 1 1 5C57328C
 P 9175 4025
@@
 $EndComp
 $Comp
-L yosino58-rescue:SK6812MINI-kbd-yosino58-rescue L4
+L yosino58-rescue:SK6812MINI L4
 U 1 1 5C57559A
 P 8675 4025
@@
 $EndComp
 $Comp
-L yosino58-rescue:SK6812MINI-kbd-yosino58-rescue L3
+L yosino58-rescue:SK6812MINI L3
 U 1 1 5C5765F4
 P 8175 4025
@@
 $EndComp
 $Comp
-L yosino58-rescue:SK6812MINI-kbd-yosino58-rescue L2
+L yosino58-rescue:SK6812MINI L2
 U 1 1 5C5787A6
 P 7675 4025
@@
 $EndComp
 $Comp
-L yosino58-rescue:SK6812MINI-kbd-yosino58-rescue L1
+L yosino58-rescue:SK6812MINI L1
 U 1 1 5C579812
 P 7175 4025
@@
 Connection ~ 9475 4225
 $Comp
-L yosino58-rescue:SK6812MINI-kbd-yosino58-rescue L7
+L yosino58-rescue:SK6812MINI L7
 U 1 1 5C5B2498
 P 7175 4575
@@
 	6975 4675 6975 4775
 $Comp
-L yosino58-rescue:SK6812MINI-kbd-yosino58-rescue L8
+L yosino58-rescue:SK6812MINI L8
 U 1 1 5C5D0C1C
 P 7675 4575
@@
 $EndComp
 $Comp
-L yosino58-rescue:SK6812MINI-kbd-yosino58-rescue L9
+L yosino58-rescue:SK6812MINI L9
 U 1 1 5C5D3BFC
 P 8175 4575
@@
 $EndComp
 $Comp
-L yosino58-rescue:SK6812MINI-kbd-yosino58-rescue L10
+L yosino58-rescue:SK6812MINI L10
 U 1 1 5C5D6BE5
 P 8675 4575
@@
 $EndComp
 $Comp
-L yosino58-rescue:SK6812MINI-kbd-yosino58-rescue L11
+L yosino58-rescue:SK6812MINI L11
 U 1 1 5C5D9BCF
 P 9175 4575
@@
 $EndComp
 $Comp
-L yosino58-rescue:SK6812MINI-kbd-yosino58-rescue L12
+L yosino58-rescue:SK6812MINI L12
 U 1 1 5C5DCBB6
 P 9675 4575
@@
 	9875 4225 10125 4225
 $Comp
-L yosino58-rescue:SK6812MINI-kbd-yosino58-rescue L18
+L yosino58-rescue:SK6812MINI L18
 U 1 1 5C62E773
 P 9675 5125
@@
 $EndComp
 $Comp
-L yosino58-rescue:SK6812MINI-kbd-yosino58-rescue L17
+L yosino58-rescue:SK6812MINI L17
 U 1 1 5C62E77A
 P 9175 5125
@@
 $EndComp
 $Comp
-L yosino58-rescue:SK6812MINI-kbd-yosino58-rescue L16
+L yosino58-rescue:SK6812MINI L16
 U 1 1 5C62E781
 P 8675 5125
@@
 $EndComp
 $Comp
-L yosino58-rescue:SK6812MINI-kbd-yosino58-rescue L15
+L yosino58-rescue:SK6812MINI L15
 U 1 1 5C62E788
 P 8175 5125
@@
 $EndComp
 $Comp
-L yosino58-rescue:SK6812MINI-kbd-yosino58-rescue L14
+L yosino58-rescue:SK6812MINI L14
 U 1 1 5C62E78F
 P 7675 5125
@@
 $EndComp
 $Comp
-L yosino58-rescue:SK6812MINI-kbd-yosino58-rescue L13
+L yosino58-rescue:SK6812MINI L13
 U 1 1 5C62E796
 P 7175 5125
@@
 	7975 5325 8375 5325
 $Comp
-L yosino58-rescue:SK6812MINI-kbd-yosino58-rescue L19
+L yosino58-rescue:SK6812MINI L19
 U 1 1 5C6EC645
 P 7175 5675
@@
 $EndComp
 $Comp
-L yosino58-rescue:SK6812MINI-kbd-yosino58-rescue L20
+L yosino58-rescue:SK6812MINI L20
 U 1 1 5C6EC64C
 P 7675 5675
@@
 $EndComp
 $Comp
-L yosino58-rescue:SK6812MINI-kbd-yosino58-rescue L21
+L yosino58-rescue:SK6812MINI L21
 U 1 1 5C6EC653
 P 8175 5675
@@
 $EndComp
 $Comp
-L yosino58-rescue:SK6812MINI-kbd-yosino58-rescue L22
+L yosino58-rescue:SK6812MINI L22
 U 1 1 5C6EC65A
 P 8675 5675
@@
 $EndComp
 $Comp
-L yosino58-rescue:SK6812MINI-kbd-yosino58-rescue L23
+L yosino58-rescue:SK6812MINI L23
 U 1 1 5C6EC661
 P 9175 5675
@@
 $EndComp
 $Comp
-L yosino58-rescue:SK6812MINI-kbd-yosino58-rescue L24
+L yosino58-rescue:SK6812MINI L24
 U 1 1 5C6EC668
 P 9675 5675
@@
 	7375 5325 7475 5325
 $Comp
-L yosino58-rescue:SK6812MINI-kbd-yosino58-rescue L29
+L yosino58-rescue:SK6812MINI L29
 U 1 1 5C7E621E
 P 9675 6225
@@
 $EndComp
 $Comp
-L yosino58-rescue:SK6812MINI-kbd-yosino58-rescue L28
+L yosino58-rescue:SK6812MINI L28
 U 1 1 5C7E6225
 P 9175 6225
@@
 $EndComp
 $Comp
-L yosino58-rescue:SK6812MINI-kbd-yosino58-rescue L27
+L yosino58-rescue:SK6812MINI L27
 U 1 1 5C7E622C
 P 8675 6225
@@
 $EndComp
 $Comp
-L yosino58-rescue:SK6812MINI-kbd-yosino58-rescue L26
+L yosino58-rescue:SK6812MINI L26
 U 1 1 5C7E6233
 P 8175 6225
@@
 $EndComp
 $Comp
-L yosino58-rescue:SK6812MINI-kbd-yosino58-rescue L25
+L yosino58-rescue:SK6812MINI L25
 U 1 1 5C7E623A
 P 7675 6225
@@
 data
 $Comp
-L yosino58-rescue:SW_PUSH-kbd-yosino58-rescue RSW1
+L yosino58-rescue:SW_PUSH RSW1
 U 1 1 5D0EC958
 P 5050 975
@@
 	1625 1125 1625 1225
 $Comp
-L yosino58-rescue:ProMicro-kbd-yosino58-rescue U2
+L yosino58-rescue:ProMicro-BLE U2
 U 1 1 5C614951
 P 2325 3250
