File: chocolate/yosino58_chocolate.sch (KiCad schematic (older format))
At the start: 110 parts, among them J0 LED, J1 TRRS, J2 OLED, J3 OLED, J4 OLED, J5 OLED, J6 OLED, P1 i2c_pin, P2 i2c_pin, SW1 SW_PUSH, SW10 SW_PUSH, SW11 SW_PUSH, SW12 SW_PUSH, SW13 SW_PUSH, SW14 SW_PUSH, SW15 SW_PUSH, SW16 SW_PUSH, SW17 SW_PUSH, SW18 SW_PUSH, SW19 SW_PUSH, SW2 SW_PUSH, SW20 SW_PUSH, SW21 SW_PUSH, SW22 SW_PUSH, SW23 SW_PUSH, SW24 SW_PUSH, SW25 SW_PUSH, SW26 SW_PUSH, SW27 SW_PUSH, SW28 SW_PUSH, SW29 SW_PUSH, SW3 SW_PUSH, SW4 SW_PUSH, SW5 SW_PUSH, SW6 SW_PUSH, SW7 SW_PUSH, SW8 SW_PUSH, SW9 SW_PUSH, U1 ProMicro, U2 ProMicro

Commit message: ソケット版追加
Parts:
- L1, L10, L11, L12, L13, L14, L15, L16, L17, L18, L19, L2, L20, L21, L22, L23, L24, L25, L26, L27, L28, L29, L3, L4, L5, L6, L7, L8, L9: footprint yosino58_chocolate:SK6812MINI_padin_rev -> yosino58_chocolate:SK6812MINI_rev
- SW29: footprint yosino58_chocolate:CherryMX_Hotswap2U_stabilizer. -> yosino58_chocolate:Choc_Hotswap2U_stabilizer
Changed lines of the file:
@@
 F 0 "SW29" H 10750 2875 50  0000 C CNN
 F 1 "SW_PUSH" H 10650 2775 50  0000 C CNN
-F 2 "yosino58_chocolate:CherryMX_Hotswap2U_stabilizer." H 10750 2925 50  0001 C CNN
+F 2 "yosino58_chocolate:Choc_Hotswap2U_stabilizer" H 10750 2925 50  0001 C CNN
 F 3 "" H 10750 2925 50  0000 C CNN
 	1    10750 2925
@@
 F 0 "L6" H 9675 4287 51  0000 C CNN
 F 1 "SK6812MINI" H 9675 4222 16  0000 C CNN
-F 2 "yosino58_chocolate:SK6812MINI_padin_rev" H 9675 4025 60  0001 C CNN
+F 2 "yosino58_chocolate:SK6812MINI_rev" H 9675 4025 60  0001 C CNN
 F 3 "" H 9675 4025 60  0001 C CNN
 	1    9675 4025
@@
 F 0 "L5" H 9175 4287 51  0000 C CNN
 F 1 "SK6812MINI" H 9175 4222 16  0000 C CNN
-F 2 "yosino58_chocolate:SK6812MINI_padin_rev" H 9175 4025 60  0001 C CNN
+F 2 "yosino58_chocolate:SK6812MINI_rev" H 9175 4025 60  0001 C CNN
 F 3 "" H 9175 4025 60  0001 C CNN
 	1    9175 4025
@@
 F 0 "L4" H 8675 4287 51  0000 C CNN
 F 1 "SK6812MINI" H 8675 4222 16  0000 C CNN
-F 2 "yosino58_chocolate:SK6812MINI_padin_rev" H 8675 4025 60  0001 C CNN
+F 2 "yosino58_chocolate:SK6812MINI_rev" H 8675 4025 60  0001 C CNN
 F 3 "" H 8675 4025 60  0001 C CNN
 	1    8675 4025
@@
 F 0 "L3" H 8175 4287 51  0000 C CNN
 F 1 "SK6812MINI" H 8175 4222 16  0000 C CNN
-F 2 "yosino58_chocolate:SK6812MINI_padin_rev" H 8175 4025 60  0001 C CNN
+F 2 "yosino58_chocolate:SK6812MINI_rev" H 8175 4025 60  0001 C CNN
 F 3 "" H 8175 4025 60  0001 C CNN
 	1    8175 4025
@@
 F 0 "L2" H 7675 4287 51  0000 C CNN
 F 1 "SK6812MINI" H 7675 4222 16  0000 C CNN
-F 2 "yosino58_chocolate:SK6812MINI_padin_rev" H 7675 4025 60  0001 C CNN
+F 2 "yosino58_chocolate:SK6812MINI_rev" H 7675 4025 60  0001 C CNN
 F 3 "" H 7675 4025 60  0001 C CNN
 	1    7675 4025
@@
 F 0 "L1" H 7175 4287 51  0000 C CNN
 F 1 "SK6812MINI" H 7175 4222 16  0000 C CNN
-F 2 "yosino58_chocolate:SK6812MINI_padin_rev" H 7175 4025 60  0001 C CNN
+F 2 "yosino58_chocolate:SK6812MINI_rev" H 7175 4025 60  0001 C CNN
 F 3 "" H 7175 4025 60  0001 C CNN
 	1    7175 4025
@@
 F 0 "L7" H 7175 4313 51  0000 C CNN
 F 1 "SK6812MINI" H 7175 4378 16  0000 C CNN
-F 2 "yosino58_chocolate:SK6812MINI_padin_rev" H 7175 4575 60  0001 C CNN
+F 2 "yosino58_chocolate:SK6812MINI_rev" H 7175 4575 60  0001 C CNN
 F 3 "" H 7175 4575 60  0001 C CNN
 	1    7175 4575
@@
 F 0 "L8" H 7675 4313 51  0000 C CNN
 F 1 "SK6812MINI" H 7675 4378 16  0000 C CNN
-F 2 "yosino58_chocolate:SK6812MINI_padin_rev" H 7675 4575 60  0001 C CNN
+F 2 "yosino58_chocolate:SK6812MINI_rev" H 7675 4575 60  0001 C CNN
 F 3 "" H 7675 4575 60  0001 C CNN
 	1    7675 4575
@@
 F 0 "L9" H 8175 4313 51  0000 C CNN
 F 1 "SK6812MINI" H 8175 4378 16  0000 C CNN
-F 2 "yosino58_chocolate:SK6812MINI_padin_rev" H 8175 4575 60  0001 C CNN
+F 2 "yosino58_chocolate:SK6812MINI_rev" H 8175 4575 60  0001 C CNN
 F 3 "" H 8175 4575 60  0001 C CNN
 	1    8175 4575
@@
 F 0 "L10" H 8675 4313 51  0000 C CNN
 F 1 "SK6812MINI" H 8675 4378 16  0000 C CNN
-F 2 "yosino58_chocolate:SK6812MINI_padin_rev" H 8675 4575 60  0001 C CNN
+F 2 "yosino58_chocolate:SK6812MINI_rev" H 8675 4575 60  0001 C CNN
 F 3 "" H 8675 4575 60  0001 C CNN
 	1    8675 4575
@@
 F 0 "L11" H 9175 4313 51  0000 C CNN
 F 1 "SK6812MINI" H 9175 4378 16  0000 C CNN
-F 2 "yosino58_chocolate:SK6812MINI_padin_rev" H 9175 4575 60  0001 C CNN
+F 2 "yosino58_chocolate:SK6812MINI_rev" H 9175 4575 60  0001 C CNN
 F 3 "" H 9175 4575 60  0001 C CNN
 	1    9175 4575
@@
 F 0 "L12" H 9675 4313 51  0000 C CNN
 F 1 "SK6812MINI" H 9675 4378 16  0000 C CNN
-F 2 "yosino58_chocolate:SK6812MINI_padin_rev" H 9675 4575 60  0001 C CNN
+F 2 "yosino58_chocolate:SK6812MINI_rev" H 9675 4575 60  0001 C CNN
 F 3 "" H 9675 4575 60  0001 C CNN
 	1    9675 4575
@@
 F 0 "L18" H 9675 5387 51  0000 C CNN
 F 1 "SK6812MINI" H 9675 5322 16  0000 C CNN
-F 2 "yosino58_chocolate:SK6812MINI_padin_rev" H 9675 5125 60  0001 C CNN
+F 2 "yosino58_chocolate:SK6812MINI_rev" H 9675 5125 60  0001 C CNN
 F 3 "" H 9675 5125 60  0001 C CNN
 	1    9675 5125
@@
 F 0 "L17" H 9175 5387 51  0000 C CNN
 F 1 "SK6812MINI" H 9175 5322 16  0000 C CNN
-F 2 "yosino58_chocolate:SK6812MINI_padin_rev" H 9175 5125 60  0001 C CNN
+F 2 "yosino58_chocolate:SK6812MINI_rev" H 9175 5125 60  0001 C CNN
 F 3 "" H 9175 5125 60  0001 C CNN
 	1    9175 5125
@@
 F 0 "L16" H 8675 5387 51  0000 C CNN
 F 1 "SK6812MINI" H 8675 5322 16  0000 C CNN
-F 2 "yosino58_chocolate:SK6812MINI_padin_rev" H 8675 5125 60  0001 C CNN
+F 2 "yosino58_chocolate:SK6812MINI_rev" H 8675 5125 60  0001 C CNN
 F 3 "" H 8675 5125 60  0001 C CNN
 	1    8675 5125
@@
 F 0 "L15" H 8175 5387 51  0000 C CNN
 F 1 "SK6812MINI" H 8175 5322 16  0000 C CNN
-F 2 "yosino58_chocolate:SK6812MINI_padin_rev" H 8175 5125 60  0001 C CNN
+F 2 "yosino58_chocolate:SK6812MINI_rev" H 8175 5125 60  0001 C CNN
 F 3 "" H 8175 5125 60  0001 C CNN
 	1    8175 5125
@@
 F 0 "L14" H 7675 5387 51  0000 C CNN
 F 1 "SK6812MINI" H 7675 5322 16  0000 C CNN
-F 2 "yosino58_chocolate:SK6812MINI_padin_rev" H 7675 5125 60  0001 C CNN
+F 2 "yosino58_chocolate:SK6812MINI_rev" H 7675 5125 60  0001 C CNN
 F 3 "" H 7675 5125 60  0001 C CNN
 	1    7675 5125
@@
 F 0 "L13" H 7175 5387 51  0000 C CNN
 F 1 "SK6812MINI" H 7175 5322 16  0000 C CNN
-F 2 "yosino58_chocolate:SK6812MINI_padin_rev" H 7175 5125 60  0001 C CNN
+F 2 "yosino58_chocolate:SK6812MINI_rev" H 7175 5125 60  0001 C CNN
 F 3 "" H 7175 5125 60  0001 C CNN
 	1    7175 5125
@@
 F 0 "L19" H 7175 5413 51  0000 C CNN
 F 1 "SK6812MINI" H 7175 5478 16  0000 C CNN
-F 2 "yosino58_chocolate:SK6812MINI_padin_rev" H 7175 5675 60  0001 C CNN
+F 2 "yosino58_chocolate:SK6812MINI_rev" H 7175 5675 60  0001 C CNN
 F 3 "" H 7175 5675 60  0001 C CNN
 	1    7175 5675
@@
 F 0 "L20" H 7675 5413 51  0000 C CNN
 F 1 "SK6812MINI" H 7675 5478 16  0000 C CNN
-F 2 "yosino58_chocolate:SK6812MINI_padin_rev" H 7675 5675 60  0001 C CNN
+F 2 "yosino58_chocolate:SK6812MINI_rev" H 7675 5675 60  0001 C CNN
 F 3 "" H 7675 5675 60  0001 C CNN
 	1    7675 5675
@@
 F 0 "L21" H 8175 5413 51  0000 C CNN
 F 1 "SK6812MINI" H 8175 5478 16  0000 C CNN
-F 2 "yosino58_chocolate:SK6812MINI_padin_rev" H 8175 5675 60  0001 C CNN
+F 2 "yosino58_chocolate:SK6812MINI_rev" H 8175 5675 60  0001 C CNN
 F 3 "" H 8175 5675 60  0001 C CNN
 	1    8175 5675
@@
 F 0 "L22" H 8675 5413 51  0000 C CNN
 F 1 "SK6812MINI" H 8675 5478 16  0000 C CNN
-F 2 "yosino58_chocolate:SK6812MINI_padin_rev" H 8675 5675 60  0001 C CNN
+F 2 "yosino58_chocolate:SK6812MINI_rev" H 8675 5675 60  0001 C CNN
 F 3 "" H 8675 5675 60  0001 C CNN
 	1    8675 5675
@@
 F 0 "L23" H 9175 5413 51  0000 C CNN
 F 1 "SK6812MINI" H 9175 5478 16  0000 C CNN
-F 2 "yosino58_chocolate:SK6812MINI_padin_rev" H 9175 5675 60  0001 C CNN
+F 2 "yosino58_chocolate:SK6812MINI_rev" H 9175 5675 60  0001 C CNN
 F 3 "" H 9175 5675 60  0001 C CNN
 	1    9175 5675
@@
 F 0 "L24" H 9675 5413 51  0000 C CNN
 F 1 "SK6812MINI" H 9675 5478 16  0000 C CNN
-F 2 "yosino58_chocolate:SK6812MINI_padin_rev" H 9675 5675 60  0001 C CNN
+F 2 "yosino58_chocolate:SK6812MINI_rev" H 9675 5675 60  0001 C CNN
 F 3 "" H 9675 5675 60  0001 C CNN
 	1    9675 5675
@@
 F 0 "L29" H 9675 6487 51  0000 C CNN
 F 1 "SK6812MINI" H 9675 6422 16  0000 C CNN
-F 2 "yosino58_chocolate:SK6812MINI_padin_rev" H 9675 6225 60  0001 C CNN
+F 2 "yosino58_chocolate:SK6812MINI_rev" H 9675 6225 60  0001 C CNN
 F 3 "" H 9675 6225 60  0001 C CNN
 	1    9675 6225
@@
 F 0 "L28" H 9175 6487 51  0000 C CNN
 F 1 "SK6812MINI" H 9175 6422 16  0000 C CNN
-F 2 "yosino58_chocolate:SK6812MINI_padin_rev" H 9175 6225 60  0001 C CNN
+F 2 "yosino58_chocolate:SK6812MINI_rev" H 9175 6225 60  0001 C CNN
 F 3 "" H 9175 6225 60  0001 C CNN
 	1    9175 6225
@@
 F 0 "L27" H 8675 6487 51  0000 C CNN
 F 1 "SK6812MINI" H 8675 6422 16  0000 C CNN
-F 2 "yosino58_chocolate:SK6812MINI_padin_rev" H 8675 6225 60  0001 C CNN
+F 2 "yosino58_chocolate:SK6812MINI_rev" H 8675 6225 60  0001 C CNN
 F 3 "" H 8675 6225 60  0001 C CNN
 	1    8675 6225
@@
 F 0 "L26" H 8175 6487 51  0000 C CNN
 F 1 "SK6812MINI" H 8175 6422 16  0000 C CNN
-F 2 "yosino58_chocolate:SK6812MINI_padin_rev" H 8175 6225 60  0001 C CNN
+F 2 "yosino58_chocolate:SK6812MINI_rev" H 8175 6225 60  0001 C CNN
 F 3 "" H 8175 6225 60  0001 C CNN
 	1    8175 6225
@@
 F 0 "L25" H 7675 6487 51  0000 C CNN
 F 1 "SK6812MINI" H 7675 6422 16  0000 C CNN
-F 2 "yosino58_chocolate:SK6812MINI_padin_rev" H 7675 6225 60  0001 C CNN
+F 2 "yosino58_chocolate:SK6812MINI_rev" H 7675 6225 60  0001 C CNN
 F 3 "" H 7675 6225 60  0001 C CNN
 	1    7675 6225
